File: hardware/usb_volume_control.kicad_pcb (KiCad board)
At the start: 4 copper layers, 100 x 70 mm, 33 parts, among them J1 AVR-PDI-6, J2 USB_C_Skt_USB2.0_16P, J3 RGB_LED, J4 CAPBTN, J5 ENC, J6 BTN, U1 AVR16DU14, U2 SN74ACT596, U3 SN74ACT596

Commit message: Finished PCB and imported to FreeCAD
Routing:
- net GND: vias 11 -> 111
Other:
- board text added: "(C)2026 Kuro68k, rev 1 GPL v3"
