File: hardware/usb_volume_control.kicad_sch (KiCad schematic)
At the start: 33 parts, among them J1 AVR-PDI-6, J2 USB_C_Skt_USB2.0_16P, J3 RGB_LED, J4 CAPBTN, J5 ENC, J6 BTN, U1 AVR16DU14, U2 SN74ACT596, U3 SN74ACT596

Commit message: Rev 2 to-do notes
Other:
- note added: "To-do: - PWM for LED brightness? - LEDs sideways? - 5V for encoder - PCB to match encoder pinout"
